File: breadboard_midi.sch (KiCad schematic (older format))
At the start: 14 parts, among them J1 MIDI IN, J2 MIDI OUT, J3 Conn_01x04, J4 Conn_01x04, U1 6N138, U2 74LVC1G125

Commit message: Tweak schematic more
Other:
- note added: "Alternate Voltage Config"
- note added: "Pin Headers"
Changed lines of the file:
@@
 EESchema Schematic File Version 4
-EELAYER 30 0
+LIBS:breadboard_midi-cache
+EELAYER 26 0
 EELAYER END
 $Descr USLetter 11000 8500
 encoding utf-8
 Sheet 1 1
-Title ""
-Date ""
-Rev ""
-Comp ""
+Title "MIDI Breadboard Breakout"
+Date "2020-09-09"
+Rev "0.1"
+Comp "Max Proskauer"
 Comment1 ""
 Comment2 ""
@@
 Wire Wire Line
 	3300 4300 3350 4300
-Text Notes 3850 3400 0    50   ~ 0
+Text Notes 5200 4800 0    50   ~ 0
     5V  3.3V\nR1 280 180\nR2 220 220\nR3 220 10\nR4 220 33
+Text Notes 6200 2250 0    100  ~ 0
+Pin Headers
+Text Notes 4950 4350 0    60   ~ 0
+Alternate Voltage Config
 $EndSCHEMATC
